Commit message: Adding driven gear

File: urdf/gripper-rollpawkit-macro.xacro (robot description, xacro)
@@ -37,5 +37,5 @@
         </geometry>
       </collision>
-            <collision>
+      <collision>
         <geometry>
           <mesh filename="package://gripper-rollpawkit/meshes/servo_plate.stl"/>
@@ -44,16 +44,9 @@
     </link>
   </xacro:macro>
-  <xacro:macro name="gear_links" params="prefix">
-    <link name="${prefix}gear_links">
+  <xacro:macro name="gear_link" params="prefix mesh">
+    <link name="${prefix}gear_link">
       <visual>
         <geometry>
-          <mesh filename="package://gripper-rollpawkit/meshes/driving_gear.stl"/>
-        </geometry>
-        <material name="white"/>
-      </visual>
-      <visual>
-        <origin xyz="0 0.0258 0" />
-        <geometry>
-          <mesh filename="package://gripper-rollpawkit/meshes/driven_gear.stl"/>
+          <mesh filename="${mesh}"/>
         </geometry>
         <material name="white"/>
@@ -61,16 +54,26 @@
       <collision>
         <geometry>
-          <mesh filename="package://gripper-rollpawkit/meshes/driving_gear.stl"/>
+          <mesh filename="${mesh}"/>
         </geometry>
       </collision>
     </link>
   </xacro:macro>
-  <xacro:macro name="gear_joints" params="prefix">
-    <joint name="${prefix}gear_joints" type="revolute">
+  <xacro:macro name="driving_gear_joint" params="prefix">
+    <joint name="${prefix}driving_gear_joint" type="revolute">
       <origin xyz="0.0172 -0.0127 0.007" rpy="0 0 0"/>
       <parent link="${prefix}base_link" />
-      <child link="${prefix}gear_links" />
+      <child link="${prefix}driving_gear_link" />
       <axis xyz="0 0 1" />
       <limit lower="-0.81" upper="0" velocity="2.0" effort="1000" />
+    </joint>
+  </xacro:macro>
+  <xacro:macro name="driven_gear_joint" params="prefix">
+    <joint name="${prefix}driven_gear_joints" type="revolute">
+      <origin xyz="0.0172 0.0127 0.007" rpy="0 0 0"/>
+      <parent link="${prefix}base_link" />
+      <child link="${prefix}driven_gear_link" />
+      <axis xyz="0 0 1" />
+      <limit lower="0" upper="0.81" velocity="2.0" effort="1000" />
+      <mimic joint="${prefix}driving_gear_joint" multiplier="-1" offset="0" />
     </joint>
   </xacro:macro>
@@ -78,6 +81,8 @@
   <xacro:macro name="gripper-rollpawkit" params="prefix">
     <xacro:base_link prefix="${prefix}"/>
-    <xacro:gear_links prefix="${prefix}"/>
-    <xacro:gear_joints prefix="${prefix}"/>
+    <xacro:gear_link prefix="${prefix}driving_" mesh="package://gripper-rollpawkit/meshes/driving_gear.stl"/>
+    <xacro:gear_link prefix="${prefix}driven_" mesh="package://gripper-rollpawkit/meshes/driven_gear.stl"/>
+    <xacro:driving_gear_joint prefix="${prefix}"/>
+    <xacro:driven_gear_joint prefix="${prefix}"/>
   </xacro:macro>
 </robot>

Commit message: URDF refactoring

File: urdf/gripper-rollpawkit-macro.xacro (robot description, xacro)
@@ -17,6 +17,6 @@
   </material>
   <xacro:property name="scale" value="1.0 1.0 1.0"/>
-  <xacro:macro name="base_link" params="prefix">
-    <link name="${prefix}base_link">
+  <xacro:macro name="base_link" params="namex">
+    <link name="${namex}">
       <visual>
         <geometry>
@@ -44,6 +44,7 @@
     </link>
   </xacro:macro>
-  <xacro:macro name="gear_link" params="prefix mesh">
-    <link name="${prefix}gear_link">
+  <!-- Gears -->
+  <xacro:macro name="gear_link" params="namex mesh">
+    <link name="${namex}">
       <visual>
         <geometry>
@@ -59,30 +60,67 @@
     </link>
   </xacro:macro>
-  <xacro:macro name="driving_gear_joint" params="prefix">
-    <joint name="${prefix}driving_gear_joint" type="revolute">
+  <xacro:macro name="gear_joint" params="namex parentx childx origin mimicx:='' lo:=0 hi:=0">
+    <joint name="${namex}" type="revolute">
+      <origin xyz="${origin}" rpy="0 0 0"/>
+      <parent link="${parentx}" />
+      <child link="${childx}" />
+      <axis xyz="0 0 1" />
+      <limit lower="${lo}" upper="${hi}" velocity="2.0" effort="1000" />
+      <xacro:if value="${mimicx != ''}">
+        <mimic joint="${mimicx}" multiplier="-1" offset="0" />
+      </xacro:if>
+    </joint>
+  </xacro:macro>
+  <!-- Gear linkage -->
+  <xacro:macro name="gear_linkage_link" params="namex mesh">
+    <link name="${namex}">
+      <visual>
+        <geometry>
+          <mesh filename="${mesh}"/>
+        </geometry>
+        <material name="white"/>
+      </visual>
+      <collision>
+        <geometry>
+          <mesh filename="${mesh}"/>
+        </geometry>
+      </collision>
+    </link>
+  </xacro:macro>
+  <xacro:macro name="gear_linkage_joint" params="namex parentx childx">
+    <joint name="${namex}" type="revolute">
       <origin xyz="0.0172 -0.0127 0.007" rpy="0 0 0"/>
-      <parent link="${prefix}base_link" />
-      <child link="${prefix}driving_gear_link" />
+      <parent link="${parentx}" />
+      <child link="${childx}" />
       <axis xyz="0 0 1" />
       <limit lower="-0.81" upper="0" velocity="2.0" effort="1000" />
     </joint>
   </xacro:macro>
-  <xacro:macro name="driven_gear_joint" params="prefix">
-    <joint name="${prefix}driven_gear_joints" type="revolute">
-      <origin xyz="0.0172 0.0127 0.007" rpy="0 0 0"/>
-      <parent link="${prefix}base_link" />
-      <child link="${prefix}driven_gear_link" />
-      <axis xyz="0 0 1" />
-      <limit lower="0" upper="0.81" velocity="2.0" effort="1000" />
-      <mimic joint="${prefix}driving_gear_joint" multiplier="-1" offset="0" />
-    </joint>
-  </xacro:macro>
   <!-- Initialization of all joints and links -->
   <xacro:macro name="gripper-rollpawkit" params="prefix">
-    <xacro:base_link prefix="${prefix}"/>
-    <xacro:gear_link prefix="${prefix}driving_" mesh="package://gripper-rollpawkit/meshes/driving_gear.stl"/>
-    <xacro:gear_link prefix="${prefix}driven_" mesh="package://gripper-rollpawkit/meshes/driven_gear.stl"/>
-    <xacro:driving_gear_joint prefix="${prefix}"/>
-    <xacro:driven_gear_joint prefix="${prefix}"/>
+    <xacro:base_link namex="${prefix}base_link"/>
+    <xacro:gear_link
+        namex="${prefix}driving_gear_link"
+        mesh="package://gripper-rollpawkit/meshes/driving_gear.stl"/>
+    <xacro:gear_joint
+        namex="${prefix}driving_gear_joint"
+        parentx="${prefix}base_link"
+        childx="${prefix}driving_gear_link"
+        origin="0.0172 -0.0127 0.007"
+        lo="-0.81"/>
+    <xacro:gear_link
+        namex="${prefix}driven_gear_link"
+        mesh="package://gripper-rollpawkit/meshes/driven_gear.stl"/>
+    <xacro:gear_joint
+        namex="${prefix}driven_gear_joint"
+        parentx="${prefix}base_link"
+        childx="${prefix}driven_gear_link"
+        origin="0.0172 0.0127 0.007"
+        hi="0.81"
+        mimicx="${prefix}driving_gear_joint"/>
+    <xacro:gear_linkage_link
+        namex="driven_linkage_link"
+        mesh="package://gripper-rollpawkit/meshes/driven_linkage.stl"/>
+    <xacro:gear_linkage_joint namex="driven_linkage_joint" parentx="driven_gear_link" childx="driven_linkage_link"/>
   </xacro:macro>
 </robot>

Commit message: Finishing gears linkages

File: urdf/gripper-rollpawkit-macro.xacro (robot description, xacro)
@@ -88,11 +88,12 @@
     </link>
   </xacro:macro>
-  <xacro:macro name="gear_linkage_joint" params="namex parentx childx">
+  <xacro:macro name="gear_linkage_joint" params="namex parentx childx origin mimicx">
     <joint name="${namex}" type="revolute">
-      <origin xyz="0.0172 -0.0127 0.007" rpy="0 0 0"/>
+      <origin xyz="${origin}" rpy="0 0 0"/>
       <parent link="${parentx}" />
       <child link="${childx}" />
       <axis xyz="0 0 1" />
       <limit lower="-0.81" upper="0" velocity="2.0" effort="1000" />
+      <mimic joint="${mimicx}" multiplier="-1" offset="0" />
     </joint>
   </xacro:macro>
@@ -122,5 +123,19 @@
         namex="driven_linkage_link"
         mesh="package://gripper-rollpawkit/meshes/driven_linkage.stl"/>
-    <xacro:gear_linkage_joint namex="driven_linkage_joint" parentx="driven_gear_link" childx="driven_linkage_link"/>
+    <xacro:gear_linkage_joint
+        namex="driven_linkage_joint"
+        parentx="base_link"
+        childx="driven_linkage_link"
+        origin="0.0356 -0.0054 0.007"
+        mimicx="${prefix}driven_gear_joint"/>
+    <xacro:gear_linkage_link
+        namex="driving_linkage_link"
+        mesh="package://gripper-rollpawkit/meshes/driven_linkage.stl"/>
+    <xacro:gear_linkage_joint
+        namex="driving_linkage_joint"
+        parentx="base_link"
+        childx="driving_linkage_link"
+        origin="0.0356 0.0054 0.007"
+        mimicx="${prefix}driving_gear_joint"/>
   </xacro:macro>
 </robot>

Commit message: Adding driving finger

File: urdf/gripper-rollpawkit-macro.xacro (robot description, xacro)
@@ -94,30 +94,75 @@
       <child link="${childx}" />
       <axis xyz="0 0 1" />
-      <limit lower="-0.81" upper="0" velocity="2.0" effort="1000" />
-      <mimic joint="${mimicx}" multiplier="-1" offset="0" />
+      <limit lower="0" upper="0.81" velocity="2.0" effort="1000" />
+      <mimic joint="${mimicx}" multiplier="1" offset="0" />
+    </joint>
+  </xacro:macro>
+  <!-- Gear linkage -->
+  <xacro:macro name="finger_link" params="namex mesh">
+    <link name="${namex}">
+      <visual>
+        <geometry>
+          <mesh filename="${mesh}"/>
+        </geometry>
+        <material name="white"/>
+      </visual>
+      <collision>
+        <geometry>
+          <mesh filename="${mesh}"/>
+        </geometry>
+      </collision>
+    </link>
+  </xacro:macro>
+  <xacro:macro name="finger_joint" params="namex parentx childx origin mimicx">
+    <joint name="${namex}" type="revolute">
+      <origin xyz="${origin}" rpy="0 0 0"/>
+      <parent link="${parentx}" />
+      <child link="${childx}" />
+      <axis xyz="0 0 1" />
+      <limit lower="0.81" upper="0" velocity="2.0" effort="1000" />
+      <mimic joint="${mimicx}" multiplier="-1" offset="0.42" />
     </joint>
   </xacro:macro>
   <!-- Initialization of all joints and links -->
   <xacro:macro name="gripper-rollpawkit" params="prefix">
-    <xacro:base_link namex="${prefix}base_link"/>
+    <xacro:base_link namex="base_link"/>
     <xacro:gear_link
-        namex="${prefix}driving_gear_link"
+        namex="driving_gear_link"
         mesh="package://gripper-rollpawkit/meshes/driving_gear.stl"/>
     <xacro:gear_joint
-        namex="${prefix}driving_gear_joint"
-        parentx="${prefix}base_link"
-        childx="${prefix}driving_gear_link"
+        namex="driving_gear_joint"
+        parentx="base_link"
+        childx="driving_gear_link"
         origin="0.0172 -0.0127 0.007"
         lo="-0.81"/>
+    <xacro:gear_linkage_link
+        namex="driving_linkage_link"
+        mesh="package://gripper-rollpawkit/meshes/driven_linkage.stl"/>
+    <xacro:gear_linkage_joint
+        namex="driving_linkage_joint"
+        parentx="base_link"
+        childx="driving_linkage_link"
+        origin="0.0356 -0.0054 0.007"
+        mimicx="driving_gear_joint"/>
+    <xacro:finger_link
+        namex="driving_finger_link"
+        mesh="package://gripper-rollpawkit/meshes/linkage.stl"/>
+    <xacro:finger_joint
+        namex="driving_finger_joint"
+        parentx="driving_gear_link"
+        childx="driving_finger_link"
+        origin="0.0308 0 0"
+        mimicx="driving_gear_joint"/>
+    <!-- -->
     <xacro:gear_link
-        namex="${prefix}driven_gear_link"
+        namex="driven_gear_link"
         mesh="package://gripper-rollpawkit/meshes/driven_gear.stl"/>
     <xacro:gear_joint
-        namex="${prefix}driven_gear_joint"
-        parentx="${prefix}base_link"
-        childx="${prefix}driven_gear_link"
+        namex="driven_gear_joint"
+        parentx="base_link"
+        childx="driven_gear_link"
         origin="0.0172 0.0127 0.007"
         hi="0.81"
-        mimicx="${prefix}driving_gear_joint"/>
+        mimicx="driving_gear_joint"/>
     <xacro:gear_linkage_link
         namex="driven_linkage_link"
@@ -127,15 +172,6 @@
         parentx="base_link"
         childx="driven_linkage_link"
-        origin="0.0356 -0.0054 0.007"
-        mimicx="${prefix}driven_gear_joint"/>
-    <xacro:gear_linkage_link
-        namex="driving_linkage_link"
-        mesh="package://gripper-rollpawkit/meshes/driven_linkage.stl"/>
-    <xacro:gear_linkage_joint
-        namex="driving_linkage_joint"
-        parentx="base_link"
-        childx="driving_linkage_link"
         origin="0.0356 0.0054 0.007"
-        mimicx="${prefix}driving_gear_joint"/>
+        mimicx="driven_gear_joint"/>
   </xacro:macro>
 </robot>

Commit message: Adding driven finger

File: urdf/gripper-rollpawkit-macro.xacro (robot description, xacro)
@@ -98,8 +98,9 @@
     </joint>
   </xacro:macro>
-  <!-- Gear linkage -->
-  <xacro:macro name="finger_link" params="namex mesh">
+  <!-- Finger linkage -->
+  <xacro:macro name="finger_link" params="namex rpyx mesh">
     <link name="${namex}">
       <visual>
+        <origin rpy="${rpyx}"/>
         <geometry>
           <mesh filename="${mesh}"/>
@@ -108,4 +109,5 @@
       </visual>
       <collision>
+        <origin rpy="${rpyx}"/>
         <geometry>
           <mesh filename="${mesh}"/>
@@ -114,5 +116,5 @@
     </link>
   </xacro:macro>
-  <xacro:macro name="finger_joint" params="namex parentx childx origin mimicx">
+  <xacro:macro name="finger_joint" params="namex parentx childx origin lo:=0 hi:=0 offset mimicx">
     <joint name="${namex}" type="revolute">
       <origin xyz="${origin}" rpy="0 0 0"/>
@@ -120,6 +122,6 @@
       <child link="${childx}" />
       <axis xyz="0 0 1" />
-      <limit lower="0.81" upper="0" velocity="2.0" effort="1000" />
-      <mimic joint="${mimicx}" multiplier="-1" offset="0.42" />
+      <limit lower="${lo}" upper="${hi}" velocity="2.0" effort="1000" />
+      <mimic joint="${mimicx}" multiplier="-1" offset="${offset}" />
     </joint>
   </xacro:macro>
@@ -147,4 +149,5 @@
     <xacro:finger_link
         namex="driving_finger_link"
+        rpyx="0 0 0"
         mesh="package://gripper-rollpawkit/meshes/linkage.stl"/>
     <xacro:finger_joint
@@ -153,4 +156,6 @@
         childx="driving_finger_link"
         origin="0.0308 0 0"
+        lo="0.81"
+        offset="0.42"
         mimicx="driving_gear_joint"/>
     <!-- -->
@@ -174,4 +179,16 @@
         origin="0.0356 0.0054 0.007"
         mimicx="driven_gear_joint"/>
+    <xacro:finger_link
+        namex="driven_finger_link"
+        rpyx="3.14 0 0"
+        mesh="package://gripper-rollpawkit/meshes/linkage.stl"/>
+    <xacro:finger_joint
+        namex="driven_finger_joint"
+        parentx="driven_gear_link"
+        childx="driven_finger_link"
+        origin="0.0308 0 0"
+        hi="0.81"
+        offset="-0.42"
+        mimicx="driven_gear_joint"/>
   </xacro:macro>
 </robot>

Commit message: Fixing naming to incorporate prefix

File: urdf/gripper-rollpawkit-macro.xacro (robot description, xacro)
@@ -1,19 +1,4 @@
 <?xml version="1.0"?>
 <robot xmlns:xacro="http://ros.org/wiki/xacro">
-  <material name="blue">
-    <color rgba="0 0 1 1"/>
-  </material>
-  <material name="red">
-    <color rgba="1 0 0 1"/>
-  </material>
-  <material name="green">
-    <color rgba="0 1 0 1"/>
-  </material>
-  <material name="black">
-    <color rgba="0 0 0 1"/>
-  </material>
-  <material name="white">
-    <color rgba="1 1 1 1"/>
-  </material>
   <xacro:property name="scale" value="1.0 1.0 1.0"/>
   <xacro:macro name="base_link" params="namex">
@@ -128,67 +113,81 @@
   <!-- Initialization of all joints and links -->
   <xacro:macro name="gripper-rollpawkit" params="prefix">
-    <xacro:base_link namex="base_link"/>
+    <xacro:property name="base_link" value="${prefix}base_link"/>
+    <xacro:property name="driving_gear_link" value="${prefix}driving_gear_link"/>
+    <xacro:property name="driving_gear_joint" value="${prefix}driving_gear_joint"/>
+    <xacro:property name="driving_linkage_link" value="${prefix}driving_linkage_link"/>
+    <xacro:property name="driving_linkage_joint" value="${prefix}driving_linkage_joint"/>
+    <xacro:property name="driving_linkage_link" value="${prefix}driving_linkage_link"/>
+    <xacro:property name="driving_finger_link" value="${prefix}driving_finger_link"/>
+    <xacro:property name="driving_finger_joint" value="${prefix}driving_finger_joint"/>
+    <xacro:property name="driven_gear_link" value="${prefix}driven_gear_link"/>
+    <xacro:property name="driven_gear_joint" value="${prefix}driven_gear_joint"/>
+    <xacro:property name="driven_linkage_link" value="${prefix}driven_linkage_link"/>
+    <xacro:property name="driven_linkage_joint" value="${prefix}driven_linkage_joint"/>
+    <xacro:property name="driven_finger_link" value="${prefix}driven_finger_link"/>
+    <xacro:property name="driven_finger_joint" value="${prefix}driven_finger_joint"/>
+    <xacro:base_link namex="${base_link}"/>
     <xacro:gear_link
-        namex="driving_gear_link"
+        namex="${driving_gear_link}"
         mesh="package://gripper-rollpawkit/meshes/driving_gear.stl"/>
     <xacro:gear_joint
-        namex="driving_gear_joint"
-        parentx="base_link"
-        childx="driving_gear_link"
+        namex="${driving_gear_joint}"
+        parentx="${base_link}"
+        childx="${driving_gear_link}"
         origin="0.0172 -0.0127 0.007"
         lo="-0.81"/>
     <xacro:gear_linkage_link
-        namex="driving_linkage_link"
+        namex="${driving_linkage_link}"
         mesh="package://gripper-rollpawkit/meshes/driven_linkage.stl"/>
     <xacro:gear_linkage_joint
-        namex="driving_linkage_joint"
-        parentx="base_link"
-        childx="driving_linkage_link"
+        namex="${driving_linkage_joint}"
+        parentx="${base_link}"
+        childx="${driving_linkage_link}"
         origin="0.0356 -0.0054 0.007"
-        mimicx="driving_gear_joint"/>
+        mimicx="${driving_gear_joint}"/>
     <xacro:finger_link
-        namex="driving_finger_link"
+        namex="${driving_finger_link}"
         rpyx="0 0 0"
         mesh="package://gripper-rollpawkit/meshes/linkage.stl"/>
     <xacro:finger_joint
-        namex="driving_finger_joint"
-        parentx="driving_gear_link"
-        childx="driving_finger_link"
+        namex="${driving_finger_joint}"
+        parentx="${driving_gear_link}"
+        childx="${driving_finger_link}"
         origin="0.0308 0 0"
         lo="0.81"
         offset="0.42"
-        mimicx="driving_gear_joint"/>
+        mimicx="${driving_gear_joint}"/>
     <!-- -->
     <xacro:gear_link
-        namex="driven_gear_link"
+        namex="${driven_gear_link}"
         mesh="package://gripper-rollpawkit/meshes/driven_gear.stl"/>
     <xacro:gear_joint
-        namex="driven_gear_joint"
-        parentx="base_link"
-        childx="driven_gear_link"
+        namex="${driven_gear_joint}"
+        parentx="${base_link}"
+        childx="${driven_gear_link}"
         origin="0.0172 0.0127 0.007"
         hi="0.81"
-        mimicx="driving_gear_joint"/>
+        mimicx="${driving_gear_joint}"/>
     <xacro:gear_linkage_link
-        namex="driven_linkage_link"
+        namex="${driven_linkage_link}"
         mesh="package://gripper-rollpawkit/meshes/driven_linkage.stl"/>
     <xacro:gear_linkage_joint
-        namex="driven_linkage_joint"
-        parentx="base_link"
-        childx="driven_linkage_link"
+        namex="${driven_linkage_joint}"
+        parentx="${base_link}"
+        childx="${driven_linkage_link}"
         origin="0.0356 0.0054 0.007"
-        mimicx="driven_gear_joint"/>
+        mimicx="${driven_gear_joint}"/>
     <xacro:finger_link
-        namex="driven_finger_link"
+        namex="${driven_finger_link}"
         rpyx="3.14 0 0"
         mesh="package://gripper-rollpawkit/meshes/linkage.stl"/>
     <xacro:finger_joint
-        namex="driven_finger_joint"
-        parentx="driven_gear_link"
-        childx="driven_finger_link"
+        namex="${driven_finger_joint}"
+        parentx="${driven_gear_link}"
+        childx="${driven_finger_link}"
         origin="0.0308 0 0"
         hi="0.81"
         offset="-0.42"
-        mimicx="driven_gear_joint"/>
+        mimicx="${driven_gear_joint}"/>
   </xacro:macro>
 </robot>

Commit message: Allowing to give a name to the gripper not just prefix

File: urdf/gripper-rollpawkit-macro.xacro (robot description, xacro)
@@ -112,19 +112,19 @@
   </xacro:macro>
   <!-- Initialization of all joints and links -->
-  <xacro:macro name="gripper-rollpawkit" params="prefix">
-    <xacro:property name="base_link" value="${prefix}base_link"/>
-    <xacro:property name="driving_gear_link" value="${prefix}driving_gear_link"/>
-    <xacro:property name="driving_gear_joint" value="${prefix}driving_gear_joint"/>
-    <xacro:property name="driving_linkage_link" value="${prefix}driving_linkage_link"/>
-    <xacro:property name="driving_linkage_joint" value="${prefix}driving_linkage_joint"/>
-    <xacro:property name="driving_linkage_link" value="${prefix}driving_linkage_link"/>
-    <xacro:property name="driving_finger_link" value="${prefix}driving_finger_link"/>
-    <xacro:property name="driving_finger_joint" value="${prefix}driving_finger_joint"/>
-    <xacro:property name="driven_gear_link" value="${prefix}driven_gear_link"/>
-    <xacro:property name="driven_gear_joint" value="${prefix}driven_gear_joint"/>
-    <xacro:property name="driven_linkage_link" value="${prefix}driven_linkage_link"/>
-    <xacro:property name="driven_linkage_joint" value="${prefix}driven_linkage_joint"/>
-    <xacro:property name="driven_finger_link" value="${prefix}driven_finger_link"/>
-    <xacro:property name="driven_finger_joint" value="${prefix}driven_finger_joint"/>
+  <xacro:macro name="gripper-rollpawkit" params="name">
+    <xacro:property name="base_link" value="${name}"/>
+    <xacro:property name="driving_gear_link" value="${name}_driving_gear_link"/>
+    <xacro:property name="driving_gear_joint" value="${name}_driving_gear_joint"/>
+    <xacro:property name="driving_linkage_link" value="${name}_driving_linkage_link"/>
+    <xacro:property name="driving_linkage_joint" value="${name}_driving_linkage_joint"/>
+    <xacro:property name="driving_linkage_link" value="${name}_driving_linkage_link"/>
+    <xacro:property name="driving_finger_link" value="${name}_driving_finger_link"/>
+    <xacro:property name="driving_finger_joint" value="${name}_driving_finger_joint"/>
+    <xacro:property name="driven_gear_link" value="${name}_driven_gear_link"/>
+    <xacro:property name="driven_gear_joint" value="${name}_driven_gear_joint"/>
+    <xacro:property name="driven_linkage_link" value="${name}_driven_linkage_link"/>
+    <xacro:property name="driven_linkage_joint" value="${name}_driven_linkage_joint"/>
+    <xacro:property name="driven_finger_link" value="${name}_driven_finger_link"/>
+    <xacro:property name="driven_finger_joint" value="${name}_driven_finger_joint"/>
     <xacro:base_link namex="${base_link}"/>
     <xacro:gear_link
